Commit message: Change the lower and upper bound of joint3 from 90 to 135.

File: src/km1_description/urdf/km1.urdf (robot description, URDF)
Before this commit: robot km1, 7 links, 6 joints
Joints:
- joint joint3: limit lower=-1.57 upper=1.57 effort=100 velocity=1 -> lower=-2.35 upper=2.35 effort=100 velocity=1
